File: pcb/usb4butia/usb4butia.kicad_pcb (KiCad board)
At the start: 2 copper layers, 88.9 x 98.5 mm, 54 parts, among them J1 USB_B, J2 RJ45, J3 RJ45, J4 RJ45, J5 RJ45, J6 RJ45, J7 RJ45, K1 AX-12, K2 CONN_3, K3 CONN_3, P1 PICkit2, P13 Bornier, P14 CONN_2, P3 CONN_2, P4 CONN_2, P5 CONN_4, P6 CONN_1, P7 CONN_1, P9 CONN_2, SW1 RST, SW2 PROG, U1 PIC18F4550, X1 20MHz

Commit message: Usb4butia 1.9 with logo
Parts:
- added ?: LOGO_BUTIA, LOGO, F.Cu at (60.3, 89.8)
- moved J4 97.8 mm to (98.1, 35.9)
- moved J5 97.8 mm to (98.1, 57.6)
- moved K3 97.8 mm to (78.5, 66.1)
- moved P13 97.8 mm to (87.4, 103.3)
- moved P14 97.8 mm to (98.4, 100.8)
- moved P9 97.8 mm to (79.5, 102.1)
- moved R10 97.8 mm to (83.8, 59.7)
- moved R11 97.8 mm to (75.9, 69.8)
- moved R6 97.8 mm to (84.0, 36.0)
- moved R9 97.8 mm to (91.9, 48.2)
- moved ? 97.8 mm to (101.7, 20.4)
- moved ? 97.8 mm to (20.9, 20.4)
- moved ? 97.8 mm to (72.9, 107.7)
- moved ? 97.8 mm to (53.3, 107.7)
- moved C1 97.8 mm to (42.7, 51.5)
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