File: pcb/puenteH/l298hn/l298hn.kicad_pcb (KiCad board)
At the start: 2 copper layers, 48.6 x 86.2 mm, 19 parts, among them K1 CONN_3, K2 CONN_3, P1 CONN_2X2, P2 PWR, P3 CONN_2, P4 CONN_2, U1 L298

Commit message: Fix capacitor problem v1.2
Parts:
- moved C1 9.00 mm to (154.0, 98.0)
Routing:
- net HK17: track 63.0 -> 129.7 mm
- net GND: track 258.4 -> 257.6 mm
Other:
- board text added: "R08082014 v1.2"
- board text removed: "R20062013 v1.1"
Changed lines of the file:
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@@
   (general
     (links 40)
-    (no_connects 0)
-    (area 118.351299 54.698899 167.297101 141.287501)
+    (no_connects 1)
+    (area 109.067601 45.432128 172.426571 141.287501)
     (thickness 1.6002)
     (drawings 7)
-    (tracks 183)
+    (tracks 191)
     (zones 0)
     (modules 19)
@@
   )
   (setup
-    (last_trace_width 0.8001)
+    (last_trace_width 0.2032)
     (user_trace_width 0.24892)
     (user_trace_width 0.50038)
@@
     (mod_text_size 1.524 1.524)
     (mod_text_width 0.3048)
-    (pad_size 16 6)
+    (pad_size 26 8)
     (pad_drill 3.85)
     (pad_to_mask_clearance 0.254)
@@
       (usegerberextensions false)
       (excludeedgelayer false)
-      (linewidth 60)
+      (linewidth 0.150000)
       (plotframeref false)
       (viasonmask false)
@@
   )
   (module C1 (layer Component)
-    (at 145.288 95.758 180)
+    (at 154 98 180)
     (descr "Condensateur e = 1 pas")
     (tags C)
@@
       (net 3 GND)
     )
-    (pad 8 thru_hole rect (at 0 -19.3) (size 16 6) (drill 3.85 (offset 0 0.5))
+    (pad 8 thru_hole rect (at 0 -19.3) (size 26 8) (drill 3.85 (offset 0 0.5))
       (layers *.Cu *.Mask F.SilkS)
       (net 3 GND)
@@
   (gr_line (start 118.5418 141.0843) (end 118.5418 54.892) (angle 90) (layer Edge.Cuts) (width 0.381))
   (gr_line (start 167.1066 54.892) (end 167.1066 141.0843) (angle 90) (layer Edge.Cuts) (width 0.381))
-  (gr_text "R20062013   v1.1" (at 158.9532 59.5884) (layer Copper)
+  (gr_text "R08082014   v1.2" (at 162.11 59.68 270) (layer Copper)
     (effects (font (size 1.432 0.524) (thickness 0.131)) (justify mirror))
   )
-  (gr_text "H-Bridge L298HN" (at 159.6644 56.8452) (layer Copper)
+  (gr_text "H-Bridge L298HN" (at 165.35 62.7 270) (layer Copper)
     (effects (font (size 1.432 1.024) (thickness 0.256)) (justify mirror))
   )
@@
   (segment (start 146.5326 85.0646) (end 146.5326 79.8703) (width 0.8001) (layer Copper) (net 2))
   (segment (start 149.479 88.011) (end 146.5326 85.0646) (width 0.8001) (layer Copper) (net 2))
+  (segment (start 156.6545 101.6) (end 156.6545 99.3845) (width 0.8001) (layer Copper) (net 3))
+  (segment (start 156.6545 99.3845) (end 155.27 98) (width 0.8001) (layer Copper) (net 3))
+  (segment (start 156.6545 99.3845) (end 155.27 98) (width 0.2032) (layer Copper) (net 3))
+  (segment (start 156.6545 101.6) (end 156.6545 100.0655) (width 0.8001) (layer Copper) (net 3))
+  (segment (start 156.1276 79.8576) (end 151.5872 79.8576) (width 0.8001) (layer Copper) (net 3))
+  (segment (start 161.11 84.84) (end 156.1276 79.8576) (width 0.8001) (layer Copper) (net 3))
+  (segment (start 161.11 95.61) (end 161.11 84.84) (width 0.8001) (layer Copper) (net 3))
+  (segment (start 156.6545 100.0655) (end 161.11 95.61) (width 0.8001) (layer Copper) (net 3))
   (via (at 122.047 97.3455) (size 1.50114) (drill 0.8001) (layers Component Copper) (net 3))
   (via (at 122.047 94.8055) (size 1.50114) (drill 0.8001) (layers Component Copper) (net 3))
@@
   (segment (start 133.8072 81.6864) (end 134.6708 82.55) (width 0.8001) (layer Component) (net 3))
   (via (at 151.5872 79.8576) (size 1.50114) (drill 0.8001) (layers Component Copper) (net 3))
-  (segment (start 156.6418 101.1555) (end 156.6418 83.8327) (width 0.7) (layer Copper) (net 3))
-  (segment (start 156.6418 83.8327) (end 152.6794 79.8703) (width 0.7) (layer Copper) (net 3))
-  (segment (start 152.6794 79.8703) (end 151.6126 79.8703) (width 0.7) (layer Copper) (net 3))
   (segment (start 140.9954 137.6807) (end 140.9954 138.7094) (width 0.8001) (layer Copper) (net 3))
   (segment (start 151.2189 138.2141) (end 151.2189 130.7846) (width 0.8001) (layer Copper) (net 3))
@@
   (segment (start 140.9954 138.7094) (end 142.113 139.827) (width 0.8001) (layer Copper) (net 3))
   (segment (start 151.2189 130.7846) (end 151.2189 126.2126) (width 0.7) (layer Copper) (net 3))
-  (segment (start 146.558 95.758) (end 146.558 96.774) (width 0.8001) (layer Copper) (net 3))
-  (segment (start 151.384 101.6) (end 156.6545 101.6) (width 0.8001) (layer Copper) (net 3))
-  (segment (start 146.558 96.774) (end 151.384 101.6) (width 0.8001) (layer Copper) (net 3))
   (segment (start 140.9954 137.6807) (end 139.6365 137.6807) (width 0.8001) (layer Copper) (net 3))
   (segment (start 122.0724 124.1679) (end 124.5362 121.7041) (width 0.8001) (layer Copper) (net 3))
@@
   (segment (start 124.5362 121.7041) (end 124.5362 117.1461) (width 0.7) (layer Copper) (net 3))
   (segment (start 124.5362 117.1461) (end 124.5262 117.1361) (width 0.7) (layer Copper) (net 3))
-  (via (at 144.018 95.758) (size 1.50114) (drill 0.8001) (layers Component Copper) (net 4))
-  (segment (start 144.018 95.758) (end 140.5255 92.2655) (width 0.8001) (layer Component) (net 4))
-  (segment (start 140.5255 92.2655) (end 122.047 92.2655) (width 0.8001) (layer Component) (net 4))
+  (segment (start 152.73 98) (end 152.73 96.44) (width 0.8001) (layer Component) (net 4))
+  (segment (start 122.047 70.353) (end 122.047 92.2655) (width 0.8001) (layer Component) (net 4))
+  (segment (start 126.61 65.79) (end 122.047 70.353) (width 0.8001) (layer Component) (net 4))
+  (segment (start 153.67 65.79) (end 126.61 65.79) (width 0.8001) (layer Component) (net 4))
+  (segment (start 157.73 69.85) (end 153.67 65.79) (width 0.8001) (layer Component) (net 4))
+  (segment (start 157.73 91.44) (end 157.73 69.85) (width 0.8001) (layer Component) (net 4))
+  (segment (start 152.73 96.44) (end 157.73 91.44) (width 0.8001) (layer Component) (net 4))
+  (segment (start 161.7345 101.6) (end 161.7345 103.4155) (width 0.8001) (layer Copper) (net 4))
+  (segment (start 143.9672 88.9272) (end 143.9672 79.8576) (width 0.8001) (layer Copper) (net 4))
+  (segment (start 147.58 92.54) (end 143.9672 88.9272) (width 0.8001) (layer Copper) (net 4))
+  (segment (start 149.43 92.54) (end 147.58 92.54) (width 0.8001) (layer Copper) (net 4))
+  (segment (start 152.73 95.84) (end 149.43 92.54) (width 0.8001) (layer Copper) (net 4))
+  (segment (start 152.73 101.6) (end 152.73 95.84) (width 0.8001) (layer Copper) (net 4))
+  (segment (start 154.84 103.71) (end 152.73 101.6) (width 0.8001) (layer Copper) (net 4))
+  (segment (start 161.44 103.71) (end 154.84 103.71) (width 0.8001) (layer Copper) (net 4))
+  (segment (start 161.7345 103.4155) (end 161.44 103.71) (width 0.8001) (layer Copper) (net 4))
+  (via (at 152.75 98) (size 1.50114) (drill 0.8001) (layers Component Copper) (net 4))
   (via (at 122.047 92.2655) (size 1.50114) (drill 0.8001) (layers Component Copper) (net 4))
-  (segment (start 144.018 95.758) (end 144.018 79.8957) (width 0.8001) (layer Copper) (net 4))
-  (segment (start 144.018 79.8957) (end 143.9926 79.8703) (width 0.8001) (layer Copper) (net 4))
-  (segment (start 143.9926 97.6376) (end 143.9926 95.7834) (width 0.8001) (layer Copper) (net 4))
-  (segment (start 161.7345 102.8065) (end 160.909 103.632) (width 0.8001) (layer Copper) (net 4))
-  (segment (start 160.909 103.632) (end 149.987 103.632) (width 0.8001) (layer Copper) (net 4))
-  (segment (start 149.987 103.632) (end 143.9926 97.6376) (width 0.8001) (layer Copper) (net 4))
-  (segment (start 161.7345 101.6) (end 161.7345 102.8065) (width 0.8001) (layer Copper) (net 4))
-  (segment (start 143.9926 95.7834) (end 144.018 95.758) (width 0.8001) (layer Copper) (net 4))
   (segment (start 153.035 108.5215) (end 147.1295 108.5215) (width 0.8001) (layer Copper) (net 5))
   (segment (start 138.9126 100.3046) (end 138.9126 79.8703) (width 0.8001) (layer Copper) (net 5))

Commit message: shield v1.3
Parts:
- moved C2 9.08 mm to (123.4, 79.1), turned to 0 degrees
Routing:
- net HK17: track 129.7 -> 77.3 mm
- net GND: track 257.6 -> 215.4 mm
- net Vcc_12: track 129.3 -> 156.3 mm
- net EnB: track 12.5 -> 31.4 mm
- net IN3: track 72.1 -> 64.7 mm
- net IN4: track 60.9 -> 54.0 mm
Other:
- board size 48.6 x 86.2 mm -> 48.6 x 68.2 mm
- board text added: "R08062015 v1.3"
- board text removed: "R08082014 v1.2"
