File: pcb/AllSenTemplate/plantilla_allsenV2.kicad_pcb (KiCad board)
At the start: 2 copper layers, 100 x 91.5 mm, 82 parts, among them J1 RJ45, K1 CONN_3, P1 CONN_6, P3 CONN_4, SW1 SW_PUSH

Commit message: fix hk17 link
Parts:
- R1 (x2): value R -> R10kΩ
- R1: value R -> R68kΩ
- R1, R2: value 10kΩ -> R10kΩ
- R2: value ID -> R1K
- R2: value ID -> R1kΩ
- R2: value ID -> R68kΩ
- R3 (x2): value R -> R120Ω
Other:
- board size 100 x 91.5 mm -> 100 x 91.7 mm
Changed lines of the file:
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@@
     (area 103.43962 49.826714 213.565378 148.39188)
     (thickness 1.6002)
-    (drawings 53)
+    (drawings 55)
     (tracks 235)
     (zones 0)
@@
       (effects (font (size 1.397 1.27) (thickness 0.2032)))
     )
-    (fp_text value R (at 0 0 270) (layer F.SilkS)
-      (effects (font (size 1.397 1.27) (thickness 0.2032)))
+    (fp_text value R120Ω (at 0 0 270) (layer F.SilkS)
+      (effects (font (size 1.197 1.07) (thickness 0.2032)))
     )
     (fp_line (start -3.81 0) (end -3.302 0) (layer F.SilkS) (width 0.3048))
@@
       (effects (font (size 1.397 1.27) (thickness 0.2032)))
     )
-    (fp_text value ID (at 0 0 90) (layer F.SilkS)
+    (fp_text value R1K (at 0 0 90) (layer F.SilkS)
       (effects (font (size 1.397 1.27) (thickness 0.2032)))
     )
@@
       (effects (font (size 1.397 1.27) (thickness 0.2032)))
     )
-    (fp_text value R (at 0 0 90) (layer F.SilkS)
+    (fp_text value R10kΩ (at 0 0 90) (layer F.SilkS)
       (effects (font (size 1.397 1.27) (thickness 0.2032)))
     )
@@
       (effects (font (size 1.397 1.27) (thickness 0.2032)))
     )
-    (fp_text value R (at 0 0 270) (layer F.SilkS)
-      (effects (font (size 1.397 1.27) (thickness 0.2032)))
+    (fp_text value R120Ω (at 0 0 270) (layer F.SilkS)
+      (effects (font (size 1.197 1.07) (thickness 0.2032)))
     )
     (fp_line (start -3.81 0) (end -3.302 0) (layer F.SilkS) (width 0.3048))
@@
       (effects (font (size 1.397 1.27) (thickness 0.2032)))
     )
-    (fp_text value ID (at 0 0 90) (layer F.SilkS)
-      (effects (font (size 1.397 1.27) (thickness 0.2032)))
+    (fp_text value R1kΩ (at 0 0 90) (layer F.SilkS)
+      (effects (font (size 1.197 1.07) (thickness 0.2032)))
     )
     (fp_line (start -3.81 0) (end -3.302 0) (layer F.SilkS) (width 0.3048))
@@
       (effects (font (size 1.397 1.27) (thickness 0.2032)))
     )
-    (fp_text value R (at 0 0 90) (layer F.SilkS)
-      (effects (font (size 1.397 1.27) (thickness 0.2032)))
+    (fp_text value R10kΩ (at 0 0 90) (layer F.SilkS)
+      (effects (font (size 1.197 1.07) (thickness 0.2032)))
     )
     (fp_line (start -3.81 0) (end -3.302 0) (layer F.SilkS) (width 0.3048))
@@
       (effects (font (size 1.397 1.27) (thickness 0.2032)))
     )
-    (fp_text value ID (at 0 0 90) (layer F.SilkS)
-      (effects (font (size 1.397 1.27) (thickness 0.2032)))
+    (fp_text value R68kΩ (at 0 0 90) (layer F.SilkS)
+      (effects (font (size 1.197 1.07) (thickness 0.2032)))
     )
     (fp_line (start -3.81 0) (end -3.302 0) (layer F.SilkS) (width 0.3048))
@@
       (effects (font (size 1.397 1.27) (thickness 0.2032)))
     )
-    (fp_text value R (at 0 0 90) (layer F.SilkS)
-      (effects (font (size 1.397 1.27) (thickness 0.2032)))
+    (fp_text value R68kΩ (at 0 0 90) (layer F.SilkS)
+      (effects (font (size 1.197 1.07) (thickness 0.2032)))
     )
     (fp_line (start -3.81 0) (end -3.302 0) (layer F.SilkS) (width 0.3048))
@@
       (effects (font (size 1.397 1.27) (thickness 0.2032)))
     )
-    (fp_text value 10kΩ (at 0 0) (layer F.SilkS)
+    (fp_text value R10kΩ (at 0 0) (layer F.SilkS)
       (effects (font (size 1.397 1.27) (thickness 0.2032)))
     )
@@
       (effects (font (size 1.397 1.27) (thickness 0.2032)))
     )
-    (fp_text value 10kΩ (at 0 0 180) (layer F.SilkS)
+    (fp_text value R10kΩ (at 0 0 180) (layer F.SilkS)
       (effects (font (size 1.397 1.27) (thickness 0.2032)))
     )
@@
     )
   )
+  (gr_line (start 148.5 63.5) (end 184.5 63.5) (angle 90) (layer Edge.Cuts) (width 0.381))
+  (gr_line (start 148.5 53) (end 148.5 63.5) (angle 90) (layer Edge.Cuts) (width 0.381))
   (gr_text "Designed in\n Uruguay" (at 188.84138 134.99084) (layer B.SilkS)
     (effects (font (size 1.03124 0.52324) (thickness 0.13208)))
